Commit message: updated v5_gazebo urdf

File: urdf/ur5_joint_limited_robot.urdf (robot description, URDF)
Before this commit: robot ur5, 44 links, 43 joints
Links:
- removed link map
- added link world
- link upper_chasis: geometry collision mesh filename=package://v5_asm/meshes/upper_chasis.STL; visual mesh filename=package://v5_asm/meshes/upper_chasis.STL
Joints:
- joint kinect: origin xyz=0.33702 0.80334 0.31779 rpy=3.1416 -1.5708 0 -> xyz=0.378055 0.80334 0.30488 rpy=-1.57079632679 -1.5708 0
- joint lidar: origin xyz=0.40469 0.76764 0.30488 rpy=3.1416 0 0.087266 -> xyz=0.40469 0.763 0.30488 rpy=1.57079632679 0 0
- joint monitor: origin xyz=0.4177 0.55518 0.3106 rpy=1.5708 1.5708 0 -> xyz=0.4177 0.55518 0.3106 rpy=0 1.5708 0
- joint world_to_base: parent map -> world
